Commit message: Added pan-tilt head collision model into simplified URDF

File: assets/devkit_base_descr.urdf (robot description, URDF)
Before this commit: robot devkit_base_descr, 15 links, 14 joints
Links:
- added link pan_tilt_base; collision mesh filename=package://dim_cpp/meshes/devkit_base/pan_tilt_base_collisio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 scale=1 1 1; visual mesh filename=package://dim_cpp/meshes/devkit_base/pan_tilt_base_collisio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 scale=1 1 1
- added link pan_tilt_head; collision mesh filename=package://dim_cpp/meshes/devkit_base/pan_tilt_head_collisio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 scale=1 1 1; visual mesh filename=package://dim_cpp/meshes/devkit_base/pan_tilt_head_collisio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 scale=1 1 1
- added link pan_tilt_pan; collision mesh filename=package://dim_cpp/meshes/devkit_base/pan_tilt_pan_collision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 scale=1 1 1; visual mesh filename=package://dim_cpp/meshes/devkit_base/pan_tilt_pan_collision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 scale=1 1 1
Joints:
- added joint pan_tilt_base_joint: type fixed, parent devkit_base_link, child pan_tilt_base, origin xyz=0 0 0 rpy=0 0 0
- added joint pan_tilt_head_joint: type revolute, parent pan_tilt_pan, child pan_tilt_head, origin xyz=0 0 1.6465 rpy=0 0 0, axis 1 0 0, limit lower=-1.57 upper=1.57 effort=100 velocity=1
- added joint pan_tilt_pan_joint: type revolute, parent pan_tilt_base, child pan_tilt_pan, origin xyz=0 .1325 0 rpy=0 0 0, axis 0 0 1, limit lower=-3.14 upper=3.14 effort=100 velocity=1

File: assets/dim_cpp/urdf/devkit_base_descr.urdf.xacro (robot description, xacro)
@@ -6,5 +6,5 @@
 	<xacro:include filename="$(find dim_cpp)/piper_description/urdf/piper_description_macro.xacro" />
 	<link name="$(arg base_frame)" />
-	<xacro:devkit_base base_frame="$(arg base_frame)" base_pos_x="0.0" base_pos_y="0.0" base_pos_z="0.0" base_roll="0.0" base_pitch="0.0" base_yaw="0.0" r="0.8" g="0.8" b="0.8" a="1.0" />
+	<xacro:devkit_base base_frame="$(arg base_frame)" base_pos_x="0.0" base_pos_y="0.0" base_pos_z="0.23625" base_roll="0.0" base_pitch="0.0" base_yaw="0.0" r="0.8" g="0.8" b="0.8" a="1.0" />
 	<xacro:piper_angled_base base_frame="pillar_platform" base_pos_x="0.0" base_pos_y="0.0" base_pos_z="0.0" base_roll="0.0" base_pitch="0.0" base_yaw="0.0" r="0.8" g="0.8" b="0.8" a="1.0" />
 	<xacro:piper_arm base_frame="piper_angled_mount" base_pos_x="0.0" base_pos_y="0.292645" base_pos_z="1.42886" base_roll="0.0" base_pitch="0.7854" base_yaw="1.5707" r="0.8" g="0.8" b="0.8" a="1.0" />

File: assets/dim_cpp/urdf/include/devkit_base.urdf.xacro (robot description, xacro)
@@ -11,9 +11,9 @@
             <parent link="${base_frame}" />
             <child link="base_center" />
-            <origin xyz="0 0 0" rpy="0 0 0" />
+            <origin xyz="${base_pos_x} ${base_pos_y} ${base_pos_z}" rpy="${base_roll} ${base_pitch} ${base_yaw}" />
         </joint>
         <link name="devkit_base_link">
             <visual>
-                <origin xyz="${base_pos_x} ${base_pos_y} ${base_pos_z}" rpy="${base_roll} ${base_pitch} ${base_yaw}" />
+                <origin xyz="0 0 0" rpy="0 0 0" />
                 <geometry>
                     <mesh filename="${file_prefix}/meshes/devkit_base/devkit_base_wheels_collision.stl" scale="1 1 1"/>
@@ -24,5 +24,5 @@
             </visual>
             <collision>
-                <origin xyz="${base_pos_x} ${base_pos_y} ${base_pos_z}" rpy="${base_roll} ${base_pitch} ${base_yaw}" />
+                <origin xyz="0 0 0" rpy="0 0 0" />
                 <geometry>
                     <mesh filename="${file_prefix}/meshes/devkit_base/devkit_base_wheels_collision.stl" scale="1 1 1"/>
@@ -42,4 +42,83 @@
             <child link="devkit_base_link" />
             <origin xyz="0 0 0" rpy="0 0 1.5707" />
+        </joint>
+        <link name="pan_tilt_base">
+            <visual>
+                <origin xyz="0 0 0" rpy="0 0 0" />
+                <geometry>
+                    <mesh filename="${file_prefix}/meshes/devkit_base/pan_tilt_base_collision.stl" scale="1 1 1"/>
+                </geometry>
+                <material name="mat">
+                    <color rgba="${r} ${g} ${b} ${a}" />
+                </material>
+            </visual>
+            <collision>
+                <origin xyz="0 0 0" rpy="0 0 0" />
+                <geometry>
+                    <mesh filename="${file_prefix}/meshes/devkit_base/pan_tilt_base_collision.stl" scale="1 1 1"/>
+                </geometry>
+                <material name="mat">
+                    <color rgba="${r} ${g} ${b} ${a}" />
+                </material>
+            </collision>
+        </link>
+        <joint name="pan_tilt_base_joint" type="fixed">
+            <parent link="devkit_base_link" />
+            <child link="pan_tilt_base" />
+            <origin xyz="0 0 0" rpy="0 0 0" />
+        </joint>
+        <link name="pan_tilt_pan">
+            <visual>
+                <origin xyz="0 -.1325 0" rpy="0 0 0" />
+                <geometry>
+                    <mesh filename="${file_prefix}/meshes/devkit_base/pan_tilt_pan_collision.stl" scale="1 1 1"/>
+                </geometry>
+                <material name="mat">
+                    <color rgba="${r} ${g} ${b} ${a}" />
+                </material>
+            </visual>
+            <collision>
+                <origin xyz="0 -.1325 0" rpy="0 0 0" />
+                <geometry>
+                    <mesh filename="${file_prefix}/meshes/devkit_base/pan_tilt_pan_collision.stl" scale="1 1 1"/>
+                </geometry>
+                <material name="mat">
+                    <color rgba="${r} ${g} ${b} ${a}" />
+                </material>
+            </collision>
+        </link>
+        <joint name="pan_tilt_pan_joint" type="revolute">
+            <parent link="pan_tilt_base" />
+            <child link="pan_tilt_pan" />
+            <origin xyz="0 .1325 0" rpy="0 0 0" />
+            <axis xyz="0 0 1" />
+            <limit lower="-3.14" upper="3.14" effort="100" velocity="1"/>
+        </joint>
+        <link name="pan_tilt_head">
+            <visual>
+                <origin xyz="0 -.1325 -1.6465" rpy="0 0 0" />
+                <geometry>
+                    <mesh filename="${file_prefix}/meshes/devkit_base/pan_tilt_head_collision.stl" scale="1 1 1"/>
+                </geometry>
+                <material name="mat">
+                    <color rgba="${r} ${g} ${b} ${a}" />
+                </material>
+            </visual>
+            <collision>
+                <origin xyz="0 -.1325 -1.6465" rpy="0 0 0" />
+                <geometry>
+                    <mesh filename="${file_prefix}/meshes/devkit_base/pan_tilt_head_collision.stl" scale="1 1 1"/>
+                </geometry>
+                <material name="mat">
+                    <color rgba="${r} ${g} ${b} ${a}" />
+                </material>
+            </collision>
+        </link>
+        <joint name="pan_tilt_head_joint" type="revolute">
+            <parent link="pan_tilt_pan" />
+            <child link="pan_tilt_head" />
+            <origin xyz="0 0 1.6465" rpy="0 0 0" />
+            <axis xyz="1 0 0" />
+            <limit lower="-1.57" upper="1.57" effort="100" velocity="1"/>
         </joint>
         <link name="pillar_platform">

Commit message: Added camera link to urdf

File: assets/devkit_base_descr.urdf (robot description, URDF)
Before this commit: robot devkit_base_descr, 18 links, 17 joints
Links:
- added link camera_center_link
Joints:
- added joint camera_center_joint: type fixed, parent pan_tilt_head, child camera_center_link, origin xyz=0 0.027 .057055 rpy=0 0 0
- joint pan_tilt_head_joint: origin xyz=0 0 1.6465 rpy=0 0 0 -> xyz=0 0 1.659 rpy=0 0 0

File: assets/dim_cpp/urdf/devkit_base_descr.urdf (robot description, URDF)
Before this commit: robot devkit_base_descr, 18 links, 17 joints
Links:
- added link camera_center_link
Joints:
- added joint camera_center_joint: type fixed, parent pan_tilt_head, child camera_center_link, origin xyz=0 0.027 .057055 rpy=0 0 0
- joint pan_tilt_head_joint: origin xyz=0 0 1.6465 rpy=0 0 0 -> xyz=0 0 1.659 rpy=0 0 0

File: assets/dim_cpp/urdf/include/devkit_base.urdf.xacro (robot description, xacro)
@@ -97,5 +97,5 @@
         <link name="pan_tilt_head">
             <visual>
-                <origin xyz="0 -.1325 -1.6465" rpy="0 0 0" />
+                <origin xyz="0 -.1325 -1.659" rpy="0 0 0" />
                 <geometry>
                     <mesh filename="${file_prefix}/meshes/devkit_base/pan_tilt_head_collision.stl" scale="1 1 1"/>
@@ -106,5 +106,5 @@
             </visual>
             <collision>
-                <origin xyz="0 -.1325 -1.6465" rpy="0 0 0" />
+                <origin xyz="0 -.1325 -1.659" rpy="0 0 0" />
                 <geometry>
                     <mesh filename="${file_prefix}/meshes/devkit_base/pan_tilt_head_collision.stl" scale="1 1 1"/>
@@ -118,7 +118,13 @@
             <parent link="pan_tilt_pan" />
             <child link="pan_tilt_head" />
-            <origin xyz="0 0 1.6465" rpy="0 0 0" />
+            <origin xyz="0 0 1.659" rpy="0 0 0" />
             <axis xyz="1 0 0" />
             <limit lower="-1.57" upper="1.57" effort="100" velocity="1"/>
+        </joint>
+        <link name="camera_center_link" />
+        <joint name="camera_center_joint" type="fixed">
+            <parent link="pan_tilt_head" />
+            <child link="camera_center_link" />
+            <origin xyz="0 0.027 .057055" rpy="0 0 0" />
         </joint>
         <link name="pillar_platform">
